File: udb-s.kicad_pcb (KiCad board)
At the start: 4 copper layers, 40 x 9 mm, 11 parts, among them J1 TYPE-C-31-M-12, J2 78171-0004, U1 TPD4E05U06DQAR

Commit message: the pcb
changed everything i wanted
Parts:
- removed G***: LOGO, locallib:UnifiedLogo
- removed U1: TPD4E05U06DQAR, acheron_Components:USON-10_2.5x1.0mm_P0.5mm
- added D2: PRTR5V0U2X, Package_TO_SOT_SMD:SOT-143, F.Cu at (127.8, 92.3)
- D1: footprint Diode_SMD:D_SOD-523 -> Diode_SMD:D_SOD-123F
- J2: footprint locallib:PicoEZMate-Reinforced-Lite -> Connector_JST:JST_SH_SM04B-SRSS-TB_1x04-1MP_P1.00mm_Horizontal
- R1, R2: footprint Resistor_SMD:R_0402_1005Metric -> Resistor_SMD:R_0805_2012Metric
- moved F1 8.87 mm to (119.8, 91.8), turned to 0 degrees
- moved D1 2.47 mm to (127.3, 96.3)
- moved R1 2.41 mm to (129.8, 96.4)
- moved R2 2.15 mm to (132.8, 96.4)
- moved FB1 1.10 mm to (132.1, 91.6), turned to 180 degrees
- moved J2 0.10 mm to (122.0, 96.4)
Routing:
- net D+: track 49.6 -> 22.3 mm, vias 5 -> 0
- net D-: track 49.5 -> 22.4 mm, vias 5 -> 0
- net GNDPWR: track 10.0 -> 18.2 mm
- net GND: track 0.43 -> 4.99 mm, vias 6 -> 5
- net Net-(J1-CC2): track 10.9 -> 7.76 mm
- net VBUS: track 29.3 -> 31.0 mm, vias 2 -> 0
- net Net-(J1-CC1): track 12.8 -> 14.3 mm
- net 5V: track 9.19 -> 8.61 mm, vias 2 -> 0
- removed copper zone on In1.Cu, net GND
- removed copper zone on In2.Cu, net GND
Other:
- copper layers 4 -> 2
- board text added: "UDB-S with the JST connector with easier to solder and bigger components"
- board text added: "i hate the molex connector"
- board text removed: "USE ONLY uDB CABLES"
- board text removed: "Unified-S1 V1.1"
- board text removed: "Unified-S1 V1.1 www.unified- daughterboard.github.io"
