File: udb-s.kicad_sch (KiCad schematic)
At the start: 10 parts, among them J1 TYPE-C-31-M-12, J2 78171-0004, U1 TPD4E05U06DQAR

Commit message: the pcb
changed everything i wanted
Parts:
- removed U1: TPD4E05U06DQAR, acheron_Components:USON-10_2.5x1.0mm_P0.5mm, symbol acheron_Symbols:TPD4E05U06DQAR
- added D2: PRTR5V0U2X, Package_TO_SOT_SMD:SOT-143, symbol Power_Protection:PRTR5V0U2X
- D1: footprint Diode_SMD:D_SOD-523 -> Diode_SMD:D_SOD-123F
- J2: footprint locallib:PicoEZMate-Reinforced-Lite -> Connector_JST:JST_SH_SM04B-SRSS-TB_1x04-1MP_P1.00mm_Horizontal
- R1, R2: footprint Resistor_SMD:R_0402_1005Metric -> Resistor_SMD:R_0805_2012Metric
Connections:
- net 5V: now also D2.4 (VCC)
- net D+: now also D2.2 (I/O1)
- net D-: now also D2.3 (I/O2)
- net GND: now also D2.1 (GND)
